File: nyak/tablo/tablo.kicad_pcb (KiCad board)
At the start: 2 copper layers, 6 parts, among them U1 74LS573, U2 ULN2803A

Commit message: more tracks
Parts:
- removed R1, R2, R3, R4: R, Resistor_THT:R_Axial_DIN0204_L3.6mm_D1.6mm_P5.08mm_Horizontal
- removed U1: 74LS573, Package_DIP:DIP-16_W7.62mm
- removed U2: ULN2803A, Package_DIP:DIP-16_W7.62mm
- added JC1: Conn_01x08_Male, Connector_PinHeader_2.54mm:PinHeader_1x08_P2.54mm_Vertical, F.Cu at (22.7, 88.6)
- added JC2: Conn_01x08_Male, Connector_PinHeader_2.54mm:PinHeader_1x08_P2.54mm_Vertical, F.Cu at (24.0, 75.9)
- added JC3: Conn_01x08_Male, Connector_PinHeader_2.54mm:PinHeader_1x08_P2.54mm_Vertical, F.Cu at (22.7, 45.4)
- added JC4: Conn_01x08_Male, Connector_PinHeader_2.54mm:PinHeader_1x08_P2.54mm_Vertical, F.Cu at (111.8, 27.9)
- added JC5: Conn_01x08_Male, Connector_PinHeader_2.54mm:PinHeader_1x08_P2.54mm_Vertical, F.Cu at (111.8, 57.1)
- added JC6: Conn_01x08_Male, Connector_PinHeader_2.54mm:PinHeader_1x08_P2.54mm_Vertical, F.Cu at (111.8, 86.4)
- added JR1: Conn_01x08_Male, Connector_PinHeader_2.54mm:PinHeader_1x08_P2.54mm_Vertical, F.Cu at (203.2, 16.5)
- added JR2: Conn_01x08_Male, Connector_PinHeader_2.54mm:PinHeader_1x08_P2.54mm_Vertical, F.Cu at (203.2, 40.6)
- added JRPI1: Conn_02x20_Odd_Even, Connector_PinSocket_2.54mm:PinSocket_2x20_P2.54mm_Vertical, B.Cu at (127.6, 25.4)
- added QR1: BD250, Package_TO_SOT_THT:TO-220-3_Vertical, F.Cu at (189.2, 17.8)
- added QR10: BD250, Package_TO_SOT_THT:TO-220-3_Vertical, F.Cu at (189.2, 63.5)
- added QR11: BD250, Package_TO_SOT_THT:TO-220-3_Vertical, F.Cu at (189.2, 68.6)
- added QR12: BD250, Package_TO_SOT_THT:TO-220-3_Vertical, F.Cu at (189.2, 73.7)
- added QR2: BD250, Package_TO_SOT_THT:TO-220-3_Vertical, F.Cu at (189.2, 22.9)
- added QR3: BD250, Package_TO_SOT_THT:TO-220-3_Vertical, F.Cu at (189.2, 27.9)
- added QR4: BD250, Package_TO_SOT_THT:TO-220-3_Vertical, F.Cu at (189.2, 33.0)
- added QR5: BD250, Package_TO_SOT_THT:TO-220-3_Vertical, F.Cu at (189.2, 38.1)
- added QR6: BD250, Package_TO_SOT_THT:TO-220-3_Vertical, F.Cu at (189.2, 43.2)
- added QR7: BD250, Package_TO_SOT_THT:TO-220-3_Vertical, F.Cu at (189.2, 48.3)
- added QR8: BD250, Package_TO_SOT_THT:TO-220-3_Vertical, F.Cu at (189.2, 53.3)
- added QR9: BD250, Package_TO_SOT_THT:TO-220-3_Vertical, F.Cu at (189.2, 58.4)
- added RC1: R, Resistor_THT:R_Axial_DIN0204_L3.6mm_D1.6mm_P7.62mm_Horizontal, F.Cu at (29.1, 106.4)
- added RC10: R, Resistor_THT:R_Axial_DIN0204_L3.6mm_D1.6mm_P7.62mm_Horizontal, F.Cu at (29.1, 73.4)
- added RC11: R, Resistor_THT:R_Axial_DIN0204_L3.6mm_D1.6mm_P7.62mm_Horizontal, F.Cu at (29.1, 70.8)
- added RC12: R, Resistor_THT:R_Axial_DIN0204_L3.6mm_D1.6mm_P7.62mm_Horizontal, F.Cu at (30.3, 68.3)
- added RC13: R, Resistor_THT:R_Axial_DIN0204_L3.6mm_D1.6mm_P7.62mm_Horizontal, F.Cu at (30.3, 65.8)
- added RC14: R, Resistor_THT:R_Axial_DIN0204_L3.6mm_D1.6mm_P7.62mm_Horizontal, F.Cu at (30.3, 63.2)
- added RC15: R, Resistor_THT:R_Axial_DIN0204_L3.6mm_D1.6mm_P7.62mm_Horizontal, F.Cu at (30.3, 60.7)
- added RC16: R, Resistor_THT:R_Axial_DIN0204_L3.6mm_D1.6mm_P7.62mm_Horizontal, F.Cu at (30.3, 58.1)
- added RC17: R, Resistor_THT:R_Axial_DIN0204_L3.6mm_D1.6mm_P7.62mm_Horizontal, F.Cu at (29.1, 45.4)
- added RC18: R, Resistor_THT:R_Axial_DIN0204_L3.6mm_D1.6mm_P7.62mm_Horizontal, F.Cu at (27.8, 42.9)
- added RC19: R, Resistor_THT:R_Axial_DIN0204_L3.6mm_D1.6mm_P7.62mm_Horizontal, F.Cu at (27.8, 40.4)
- added RC2: R, Resistor_THT:R_Axial_DIN0204_L3.6mm_D1.6mm_P7.62mm_Horizontal, F.Cu at (29.1, 103.9)
- added RC20: R, Resistor_THT:R_Axial_DIN0204_L3.6mm_D1.6mm_P7.62mm_Horizontal, F.Cu at (27.8, 37.8)
- added RC21: R, Resistor_THT:R_Axial_DIN0204_L3.6mm_D1.6mm_P7.62mm_Horizontal, F.Cu at (27.8, 35.3)
- added RC22: R, Resistor_THT:R_Axial_DIN0204_L3.6mm_D1.6mm_P7.62mm_Horizontal, F.Cu at (27.8, 32.7)
- added RC23: R, Resistor_THT:R_Axial_DIN0204_L3.6mm_D1.6mm_P7.62mm_Horizontal, F.Cu at (27.8, 30.2)
- added RC24: R, Resistor_THT:R_Axial_DIN0204_L3.6mm_D1.6mm_P7.62mm_Horizontal, F.Cu at (27.8, 27.7)
- added RC25: R, Resistor_THT:R_Axial_DIN0204_L3.6mm_D1.6mm_P7.62mm_Horizontal, F.Cu at (108.0, 27.9)
- added RC26: R, Resistor_THT:R_Axial_DIN0204_L3.6mm_D1.6mm_P7.62mm_Horizontal, F.Cu at (108.0, 30.5)
- added RC27: R, Resistor_THT:R_Axial_DIN0204_L3.6mm_D1.6mm_P7.62mm_Horizontal, F.Cu at (108.0, 33.0)
- added RC28: R, Resistor_THT:R_Axial_DIN0204_L3.6mm_D1.6mm_P7.62mm_Horizontal, F.Cu at (108.0, 35.6)
- added RC29: R, Resistor_THT:R_Axial_DIN0204_L3.6mm_D1.6mm_P7.62mm_Horizontal, F.Cu at (108.0, 38.1)
- added RC3: R, Resistor_THT:R_Axial_DIN0204_L3.6mm_D1.6mm_P7.62mm_Horizontal, F.Cu at (29.1, 101.3)
- added RC30: R, Resistor_THT:R_Axial_DIN0204_L3.6mm_D1.6mm_P7.62mm_Horizontal, F.Cu at (108.0, 40.6)
- added RC31: R, Resistor_THT:R_Axial_DIN0204_L3.6mm_D1.6mm_P7.62mm_Horizontal, F.Cu at (108.0, 43.2)
- added RC32: R, Resistor_THT:R_Axial_DIN0204_L3.6mm_D1.6mm_P7.62mm_Horizontal, F.Cu at (108.0, 45.7)
- added RC33: R, Resistor_THT:R_Axial_DIN0204_L3.6mm_D1.6mm_P7.62mm_Horizontal, F.Cu at (108.0, 57.1)
- added RC34: R, Resistor_THT:R_Axial_DIN0204_L3.6mm_D1.6mm_P7.62mm_Horizontal, F.Cu at (108.0, 59.7)
- added RC35: R, Resistor_THT:R_Axial_DIN0204_L3.6mm_D1.6mm_P7.62mm_Horizontal, F.Cu at (108.0, 62.2)
- added RC36: R, Resistor_THT:R_Axial_DIN0204_L3.6mm_D1.6mm_P7.62mm_Horizontal, F.Cu at (108.0, 64.8)
- added RC37: R, Resistor_THT:R_Axial_DIN0204_L3.6mm_D1.6mm_P7.62mm_Horizontal, F.Cu at (108.0, 67.3)
- added RC38: R, Resistor_THT:R_Axial_DIN0204_L3.6mm_D1.6mm_P7.62mm_Horizontal, F.Cu at (108.0, 69.8)
- added RC39: R, Resistor_THT:R_Axial_DIN0204_L3.6mm_D1.6mm_P7.62mm_Horizontal, F.Cu at (108.0, 72.4)
- added RC4: R, Resistor_THT:R_Axial_DIN0204_L3.6mm_D1.6mm_P7.62mm_Horizontal, F.Cu at (29.1, 98.8)
- added RC40: R, Resistor_THT:R_Axial_DIN0204_L3.6mm_D1.6mm_P7.62mm_Horizontal, F.Cu at (108.0, 74.9)
- added RC41: R, Resistor_THT:R_Axial_DIN0204_L3.6mm_D1.6mm_P7.62mm_Horizontal, F.Cu at (108.0, 86.4)
- added RC42: R, Resistor_THT:R_Axial_DIN0204_L3.6mm_D1.6mm_P7.62mm_Horizontal, F.Cu at (108.0, 88.9)
- added RC43: R, Resistor_THT:R_Axial_DIN0204_L3.6mm_D1.6mm_P7.62mm_Horizontal, F.Cu at (108.0, 91.4)
- added RC44: R, Resistor_THT:R_Axial_DIN0204_L3.6mm_D1.6mm_P7.62mm_Horizontal, F.Cu at (108.0, 94.0)
- added RC45: R, Resistor_THT:R_Axial_DIN0204_L3.6mm_D1.6mm_P7.62mm_Horizontal, F.Cu at (108.0, 96.5)
- added RC46: R, Resistor_THT:R_Axial_DIN0204_L3.6mm_D1.6mm_P7.62mm_Horizontal, F.Cu at (108.0, 99.1)
- added RC47: R, Resistor_THT:R_Axial_DIN0204_L3.6mm_D1.6mm_P7.62mm_Horizontal, F.Cu at (108.0, 101.6)
- added RC48: R, Resistor_THT:R_Axial_DIN0204_L3.6mm_D1.6mm_P7.62mm_Horizontal, F.Cu at (108.0, 104.1)
- added RC5: R, Resistor_THT:R_Axial_DIN0204_L3.6mm_D1.6mm_P7.62mm_Horizontal, F.Cu at (29.1, 96.2)
- added RC6: R, Resistor_THT:R_Axial_DIN0204_L3.6mm_D1.6mm_P7.62mm_Horizontal, F.Cu at (29.1, 93.7)
- added RC7: R, Resistor_THT:R_Axial_DIN0204_L3.6mm_D1.6mm_P7.62mm_Horizontal, F.Cu at (29.1, 91.2)
- added RC8: R, Resistor_THT:R_Axial_DIN0204_L3.6mm_D1.6mm_P7.62mm_Horizontal, F.Cu at (29.1, 88.6)
- added RC9: R, Resistor_THT:R_Axial_DIN0204_L3.6mm_D1.6mm_P7.62mm_Horizontal, F.Cu at (29.1, 75.9)
- added RRB1: R, Resistor_THT:R_Axial_DIN0204_L3.6mm_D1.6mm_P7.62mm_Horizontal, F.Cu at (179.1, 17.8)
- added RRB10: R, Resistor_THT:R_Axial_DIN0204_L3.6mm_D1.6mm_P7.62mm_Horizontal, F.Cu at (179.1, 63.5)
- added RRB11: R, Resistor_THT:R_Axial_DIN0204_L3.6mm_D1.6mm_P7.62mm_Horizontal, F.Cu at (179.1, 68.6)
- added RRB12: R, Resistor_THT:R_Axial_DIN0204_L3.6mm_D1.6mm_P7.62mm_Horizontal, F.Cu at (179.1, 73.7)
- added RRB2: R, Resistor_THT:R_Axial_DIN0204_L3.6mm_D1.6mm_P7.62mm_Horizontal, F.Cu at (179.1, 22.9)
- added RRB3: R, Resistor_THT:R_Axial_DIN0204_L3.6mm_D1.6mm_P7.62mm_Horizontal, F.Cu at (179.1, 27.9)
- added RRB4: R, Resistor_THT:R_Axial_DIN0204_L3.6mm_D1.6mm_P7.62mm_Horizontal, F.Cu at (179.1, 33.0)
- added RRB5: R, Resistor_THT:R_Axial_DIN0204_L3.6mm_D1.6mm_P7.62mm_Horizontal, F.Cu at (179.1, 38.1)
- added RRB6: R, Resistor_THT:R_Axial_DIN0204_L3.6mm_D1.6mm_P7.62mm_Horizontal, F.Cu at (179.1, 43.2)
- added RRB7: R, Resistor_THT:R_Axial_DIN0204_L3.6mm_D1.6mm_P7.62mm_Horizontal, F.Cu at (179.1, 48.3)
- added RRB8: R, Resistor_THT:R_Axial_DIN0204_L3.6mm_D1.6mm_P7.62mm_Horizontal, F.Cu at (179.1, 53.3)
- added RRB9: R, Resistor_THT:R_Axial_DIN0204_L3.6mm_D1.6mm_P7.62mm_Horizontal, F.Cu at (179.1, 58.4)
- added RRE1: R, Resistor_THT:R_Axial_DIN0204_L3.6mm_D1.6mm_P7.62mm_Horizontal, F.Cu at (194.3, 15.2)
- added RRE10: R, Resistor_THT:R_Axial_DIN0204_L3.6mm_D1.6mm_P7.62mm_Horizontal, F.Cu at (194.3, 61.0)
- added RRE11: R, Resistor_THT:R_Axial_DIN0204_L3.6mm_D1.6mm_P7.62mm_Horizontal, F.Cu at (194.3, 66.0)
- added RRE12: R, Resistor_THT:R_Axial_DIN0204_L3.6mm_D1.6mm_P7.62mm_Horizontal, F.Cu at (194.3, 71.1)
- added RRE2: R, Resistor_THT:R_Axial_DIN0204_L3.6mm_D1.6mm_P7.62mm_Horizontal, F.Cu at (194.3, 20.3)
- added RRE3: R, Resistor_THT:R_Axial_DIN0204_L3.6mm_D1.6mm_P7.62mm_Horizontal, F.Cu at (194.3, 25.4)
- added RRE4: R, Resistor_THT:R_Axial_DIN0204_L3.6mm_D1.6mm_P7.62mm_Horizontal, F.Cu at (194.3, 30.5)
- added RRE5: R, Resistor_THT:R_Axial_DIN0204_L3.6mm_D1.6mm_P7.62mm_Horizontal, F.Cu at (194.3, 35.6)
- added RRE6: R, Resistor_THT:R_Axial_DIN0204_L3.6mm_D1.6mm_P7.62mm_Horizontal, F.Cu at (194.3, 40.6)
- added RRE7: R, Resistor_THT:R_Axial_DIN0204_L3.6mm_D1.6mm_P7.62mm_Horizontal, F.Cu at (194.3, 45.7)
- added RRE8: R, Resistor_THT:R_Axial_DIN0204_L3.6mm_D1.6mm_P7.62mm_Horizontal, F.Cu at (194.3, 50.8)
- added RRE9: R, Resistor_THT:R_Axial_DIN0204_L3.6mm_D1.6mm_P7.62mm_Horizontal, F.Cu at (194.3, 55.9)
- added UC1: ULN2803A, Package_DIP:DIP-18_W7.62mm, F.Cu at (48.1, 106.4)
- added UC2: ULN2803A, Package_DIP:DIP-18_W7.62mm, F.Cu at (48.1, 75.9)
- added UC3: ULN2803A, Package_DIP:DIP-18_W7.62mm, F.Cu at (46.8, 45.4)
- added UC4: ULN2803A, Package_DIP:DIP-18_W7.62mm, F.Cu at (89.5, 27.9)
- added UC5: ULN2803A, Package_DIP:DIP-18_W7.62mm, F.Cu at (89.5, 57.1)
- added UC6: ULN2803A, Package_DIP:DIP-18_W7.62mm, F.Cu at (89.5, 86.4)
- added UDM1: 74LS138, Package_DIP:DIP-16_W7.62mm, F.Cu at (149.9, 40.6)
- added UDM2: 74LS138, Package_DIP:DIP-16_W7.62mm, F.Cu at (151.1, 16.5)
- added UL1: 74LS573, Package_DIP:DIP-20_W7.62mm, F.Cu at (60.8, 108.9)
- added UL2: 74LS573, Package_DIP:DIP-20_W7.62mm, F.Cu at (60.8, 78.5)
- added UL3: 74LS573, Package_DIP:DIP-20_W7.62mm, F.Cu at (59.7, 48.3)
- added UL4: 74LS573, Package_DIP:DIP-20_W7.62mm, F.Cu at (78.1, 25.4)
- added UL5: 74LS573, Package_DIP:DIP-20_W7.62mm, F.Cu at (78.1, 54.6)
- added UL6: 74LS573, Package_DIP:DIP-20_W7.62mm, F.Cu at (78.1, 83.8)
- added UOD1: 74LCX07, Package_DIP:DIP-14_W7.62mm, F.Cu at (163.8, 17.8)
- added UOD2: 74LCX07, Package_DIP:DIP-14_W7.62mm, F.Cu at (163.8, 40.6)
Routing:
- net /C2: track 0.00 -> 216.4 mm, vias 0 -> 4
- net /C3: track 0.00 -> 213.8 mm, vias 0 -> 4
- net /C4: track 0.00 -> 203.2 mm, vias 0 -> 5
- net /C5: track 0.00 -> 196.0 mm, vias 0 -> 5
- net /C1: track 0.00 -> 193.7 mm, vias 0 -> 3
- net /C6: track 0.00 -> 188.1 mm, vias 0 -> 5
- net /C7: track 0.00 -> 182.6 mm, vias 0 -> 3
- net /C8: track 0.00 -> 182.3 mm, vias 0 -> 3
- net Net-(U1-Pad16): track 8.89 -> 0.00 mm
- net Net-(U1-Pad15): track 8.89 -> 0.00 mm
- net Net-(U1-Pad14): track 8.89 -> 0.00 mm
- net Net-(U1-Pad13): track 8.89 -> 0.00 mm
- net Net-(U1-Pad12): track 8.89 -> 0.00 mm
- net Net-(R4-Pad1): track 6.36 -> 0.00 mm
- net Net-(UC6-Pad8): track 0.00 -> 3.81 mm
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
Commit message: more pcb
Parts:
- moved JR1 94.6 mm to (176.5, 107.3), turned to 270 degrees
- moved JR2 93.8 mm to (137.2, 107.3), turned to 270 degrees
- moved RRE1 87.3 mm to (177.8, 101.0), turned to 90 degrees
- moved RRE2 83.5 mm to (172.7, 101.0), turned to 90 degrees
- moved RRE3 80.1 mm to (167.6, 101.0), turned to 90 degrees
- moved RRE12 78.3 mm to (121.9, 101.0), turned to 90 degrees
- moved RRE4 77.3 mm to (162.6, 101.0), turned to 90 degrees
- moved QR1 76.8 mm to (175.3, 93.3), turned to 270 degrees
- moved RRE11 75.8 mm to (127.0, 101.0), turned to 90 degrees
- moved RRE5 75.1 mm to (157.5, 101.0), turned to 90 degrees
- moved RRE10 74.0 mm to (132.1, 101.0), turned to 90 degrees
- moved RRE6 73.5 mm to (152.4, 101.0), turned to 90 degrees
- moved QR2 73.0 mm to (170.2, 93.3), turned to 270 degrees
- moved RRE9 72.8 mm to (137.2, 101.0), turned to 90 degrees
- moved QR12 72.6 mm to (119.4, 93.3), turned to 270 degrees
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Connections:
- UL1 pad 10: Net-(UL1-Pad10) -> Earth
Routing:
- net Earth: track 0.00 -> 523.5 mm
- net VCC: track 0.00 -> 382.3 mm
- net Net-(JRPI1-Pad16): track 0.00 -> 205.2 mm, vias 0 -> 4
- net /GPIO14: track 0.00 -> 100.5 mm
- net /C1: track 193.7 -> 279.7 mm, vias 3 -> 4
- net /C2: track 216.4 -> 299.2 mm, vias 4 -> 5
- net /C3: track 213.8 -> 293.1 mm, vias 4 -> 5
- net /C4: track 203.2 -> 279.7 mm, vias 5 -> 6
- net /C5: track 196.0 -> 269.7 mm, vias 5 -> 6
- net /C7: track 182.6 -> 253.0 mm, vias 3 -> 6
- net /C6: track 188.1 -> 257.9 mm, vias 5 -> 6
- net Net-(UDM2-Pad15): track 0.00 -> 69.5 mm, vias 0 -> 1
- net Net-(UDM2-Pad10): track 0.00 -> 63.6 mm, vias 0 -> 1
- net /AR2: track 0.00 -> 60.4 mm, vias 0 -> 1
- net Net-(UDM2-Pad7): track 0.00 -> 60.3 mm, vias 0 -> 2
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
Commit message: seems to be finished
Parts:
- added JTAP1: Conn_01x02_Male, Connector_PinHeader_2.54mm:PinHeader_1x02_P2.54mm_Vertical, F.Cu at (166.4, 64.1)
- moved RC3 10.6 mm to (26.7, 111.8)
- moved RC44 10.6 mm to (104.8, 106.7)
- moved RC46 10.6 mm to (104.8, 111.8)
- moved RC5 10.6 mm to (26.7, 106.7)
- moved UL2 10.6 mm to (56.5, 88.9)
- moved JRPI1 10.6 mm to (124.5, 35.6)
- moved JC3 10.6 mm to (22.9, 55.9)
- moved JC4 10.6 mm to (108.6, 38.1)
- moved RC15 10.6 mm to (26.7, 71.1)
- moved RC17 10.6 mm to (26.7, 55.9)
- moved RC18 10.6 mm to (26.7, 53.3)
- moved RC31 10.6 mm to (104.8, 53.3)
- moved RC32 10.6 mm to (104.8, 55.9)
- moved RC34 10.6 mm to (104.8, 71.1)
- moved UC3 10.6 mm to (45.1, 55.9)
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Connections:
- JRPI1 pad 2: Net-(JRPI1-Pad2) -> VCC
- JRPI1 pad 6: Net-(JRPI1-Pad6) -> Earth
Routing:
- net Earth: track 523.5 -> 671.6 mm
- net VCC: track 382.3 -> 518.7 mm
- net /GPIO17: track 0.00 -> 105.1 mm, vias 0 -> 2
- net /GPIO13: track 0.00 -> 104.0 mm, vias 0 -> 2
- net /GPIO12: track 0.00 -> 94.3 mm, vias 0 -> 2
- net /GPIO16: track 0.00 -> 48.7 mm
Other:
- board outline added: 163.8 x 106.7 mm
